Commit message: burger_vision addition.

File: turtlebot3_description/urdf/turtlebot3_burger_vision.gazebo.xacro (robot description, xacro)
@@ -124,124 +124,124 @@
     </sensor>
   </gazebo>
-  <gazebo reference="camera_link">
-    <sensor name="camera_link_camera" type="depth">
-      <update_rate>20</update_rate>
-      <camera>
-        <horizontal_fov>1.047198</horizontal_fov>
+<!--  <gazebo reference="camera_link">-->
+<!--    <sensor name="camera_link_camera" type="depth">-->
+<!--      <update_rate>20</update_rate>-->
+<!--      <camera>-->
+<!--        <horizontal_fov>1.047198</horizontal_fov>-->
+<!--        <image>-->
+<!--          <width>640</width>-->
+<!--          <height>480</height>-->
+<!--          <format>R8G8B8</format>-->
+<!--        </image>-->
+<!--        <clip>-->
+<!--          <near>0.05</near>-->
+<!--          <far>50</far>-->
+<!--        </clip>-->
+<!--      </camera>-->
+<!--      <plugin name="camera_link_controller" filename="libgazebo_ros_openni_kinect.so">-->
+<!--        <baseline>0.2</baseline>-->
+<!--        <alwaysOn>true</alwaysOn>-->
+<!--        <updateRate>1.0</updateRate>-->
+<!--        <cameraName>kinect_ir</cameraName>-->
+<!--        <imageTopicName>/kinect/color/image_raw</imageTopicName>-->
+<!--        <cameraInfoTopicName>/kinect/color/camera_info</cameraInfoTopicName>-->
+<!--        <depthImageTopicName>/kinect/depth/image_raw</depthImageTopicName>-->
+<!--        <depthImageInfoTopicName>/kinect/depth/camera_info</depthImageInfoTopicName>-->
+<!--        <pointCloudTopicName>/kinect/depth/points</pointCloudTopicName>-->
+<!--        <frameName>camera_optical_link</frameName>-->
+<!--        <pointCloudCutoff>0.5</pointCloudCutoff>-->
+<!--        <pointCloudCutoffMax>3.0</pointCloudCutoffMax>-->
+<!--        <distortionK1>0.00000001</distortionK1>-->
+<!--        <distortionK2>0.00000001</distortionK2>-->
+<!--        <distortionK3>0.00000001</distortionK3>-->
+<!--        <distortionT1>0.00000001</distortionT1>-->
+<!--        <distortionT2>0.00000001</distortionT2>-->
+<!--        <CxPrime>0</CxPrime>-->
+<!--        <Cx>0</Cx>-->
+<!--        <Cy>0</Cy>-->
+<!--        <focalLength>0</focalLength>-->
+<!--        <hackBaseline>0</hackBaseline>-->
+<!--      </plugin>-->
+<!--    </sensor>-->
+<!--  </gazebo>-->
+  <!-- camera -->
+  <gazebo reference="camera_link_left">
+    <sensor type="camera" name="camera1">
+      <update_rate>30.0</update_rate>
+      <camera name="head">
+        <horizontal_fov>1.3962634</horizontal_fov>
         <image>
-          <width>640</width>
-          <height>480</height>
+          <width>800</width>
+          <height>800</height>
           <format>R8G8B8</format>
         </image>
         <clip>
-          <near>0.05</near>
-          <far>3</far>
+          <near>0.02</near>
+          <far>300</far>
         </clip>
+        <noise>
+          <type>gaussian</type>
+          <!-- Noise is sampled independently per pixel on each frame.
+               That pixel's noise value is added to each of its color
+               channels, which at that point lie in the range [0,1]. -->
+          <mean>0.0</mean>
+          <stddev>0.007</stddev>
+        </noise>
       </camera>
-      <plugin name="camera_link_controller" filename="libgazebo_ros_openni_kinect.so">
-        <baseline>0.2</baseline>
+      <plugin name="camera_controller" filename="libgazebo_ros_camera.so">
         <alwaysOn>true</alwaysOn>
-        <updateRate>1.0</updateRate>
-        <cameraName>kinect_ir</cameraName>
-        <imageTopicName>/kinect/color/image_raw</imageTopicName>
-        <cameraInfoTopicName>/kinect/color/camera_info</cameraInfoTopicName>
-        <depthImageTopicName>/kinect/depth/image_raw</depthImageTopicName>
-        <depthImageInfoTopicName>/kinect/depth/camera_info</depthImageInfoTopicName>
-        <pointCloudTopicName>/kinect/depth/points</pointCloudTopicName>
-        <frameName>camera_optical_link</frameName>
-        <pointCloudCutoff>0.5</pointCloudCutoff>
-        <pointCloudCutoffMax>3.0</pointCloudCutoffMax>
-        <distortionK1>0.00000001</distortionK1>
-        <distortionK2>0.00000001</distortionK2>
-        <distortionK3>0.00000001</distortionK3>
-        <distortionT1>0.00000001</distortionT1>
-        <distortionT2>0.00000001</distortionT2>
-        <CxPrime>0</CxPrime>
-        <Cx>0</Cx>
-        <Cy>0</Cy>
-        <focalLength>0</focalLength>
-        <hackBaseline>0</hackBaseline>
+        <updateRate>0.0</updateRate>
+        <cameraName>stereo/left</cameraName>
+        <imageTopicName>image_raw</imageTopicName>
+        <cameraInfoTopicName>camera_info</cameraInfoTopicName>
+        <frameName>camera_link_left</frameName>
+        <hackBaseline>0.07</hackBaseline>
+        <distortionK1>0.0</distortionK1>
+        <distortionK2>0.0</distortionK2>
+        <distortionK3>0.0</distortionK3>
+        <distortionT1>0.0</distortionT1>
+        <distortionT2>0.0</distortionT2>
       </plugin>
     </sensor>
   </gazebo>
-<!--  &lt;!&ndash; camera &ndash;&gt;-->
-<!--  <gazebo reference="camera_link_left">-->
-<!--    <sensor type="camera" name="camera1">-->
-<!--      <update_rate>30.0</update_rate>-->
-<!--      <camera name="head">-->
-<!--        <horizontal_fov>1.3962634</horizontal_fov>-->
-<!--        <image>-->
-<!--          <width>800</width>-->
-<!--          <height>800</height>-->
-<!--          <format>R8G8B8</format>-->
-<!--        </image>-->
-<!--        <clip>-->
-<!--          <near>0.02</near>-->
-<!--          <far>300</far>-->
-<!--        </clip>-->
-<!--        <noise>-->
-<!--          <type>gaussian</type>-->
-<!--          &lt;!&ndash; Noise is sampled independently per pixel on each frame.-->
-<!--               That pixel's noise value is added to each of its color-->
-<!--               channels, which at that point lie in the range [0,1]. &ndash;&gt;-->
-<!--          <mean>0.0</mean>-->
-<!--          <stddev>0.007</stddev>-->
-<!--        </noise>-->
-<!--      </camera>-->
-<!--      <plugin name="camera_controller" filename="libgazebo_ros_camera.so">-->
-<!--        <alwaysOn>true</alwaysOn>-->
-<!--        <updateRate>0.0</updateRate>-->
-<!--        <cameraName>stereo/left</cameraName>-->
-<!--        <imageTopicName>image_raw</imageTopicName>-->
-<!--        <cameraInfoTopicName>camera_info</cameraInfoTopicName>-->
-<!--        <frameName>camera_link_left</frameName>-->
-<!--        <hackBaseline>0.07</hackBaseline>-->
-<!--        <distortionK1>0.0</distortionK1>-->
-<!--        <distortionK2>0.0</distortionK2>-->
-<!--        <distortionK3>0.0</distortionK3>-->
-<!--        <distortionT1>0.0</distortionT1>-->
-<!--        <distortionT2>0.0</distortionT2>-->
-<!--      </plugin>-->
-<!--    </sensor>-->
-<!--  </gazebo>-->
-<!--  &lt;!&ndash; camera &ndash;&gt;-->
-<!--  <gazebo reference="camera_link_right">-->
-<!--    <sensor type="camera" name="camera2">-->
-<!--      <update_rate>30.0</update_rate>-->
-<!--      <camera name="head">-->
-<!--        <horizontal_fov>1.3962634</horizontal_fov>-->
-<!--        <image>-->
-<!--          <width>800</width>-->
-<!--          <height>800</height>-->
-<!--          <format>R8G8B8</format>-->
-<!--        </image>-->
-<!--        <clip>-->
-<!--          <near>0.02</near>-->
-<!--          <far>300</far>-->
-<!--        </clip>-->
-<!--        <noise>-->
-<!--          <type>gaussian</type>-->
-<!--          &lt;!&ndash; Noise is sampled independently per pixel on each frame.-->
-<!--               That pixel's noise value is added to each of its color-->
-<!--               channels, which at that point lie in the range [0,1]. &ndash;&gt;-->
-<!--          <mean>0.0</mean>-->
-<!--          <stddev>0.007</stddev>-->
-<!--        </noise>-->
-<!--      </camera>-->
-<!--      <plugin name="camera_controller" filename="libgazebo_ros_camera.so">-->
-<!--        <alwaysOn>true</alwaysOn>-->
-<!--        <updateRate>0.0</updateRate>-->
-<!--        <cameraName>stereo/right</cameraName>-->
-<!--        <imageTopicName>image_raw</imageTopicName>-->
-<!--        <cameraInfoTopicName>camera_info</cameraInfoTopicName>-->
-<!--        <frameName>camera_link_right</frameName>-->
-<!--        <hackBaseline>0.07</hackBaseline>-->
-<!--        <distortionK1>0.0</distortionK1>-->
-<!--        <distortionK2>0.0</distortionK2>-->
-<!--        <distortionK3>0.0</distortionK3>-->
-<!--        <distortionT1>0.0</distortionT1>-->
-<!--        <distortionT2>0.0</distortionT2>-->
-<!--      </plugin>-->
-<!--    </sensor>-->
-<!--  </gazebo>-->
+  <!-- camera -->
+  <gazebo reference="camera_link_right">
+    <sensor type="camera" name="camera2">
+      <update_rate>30.0</update_rate>
+      <camera name="head">
+        <horizontal_fov>1.3962634</horizontal_fov>
+        <image>
+          <width>800</width>
+          <height>800</height>
+          <format>R8G8B8</format>
+        </image>
+        <clip>
+          <near>0.02</near>
+          <far>300</far>
+        </clip>
+        <noise>
+          <type>gaussian</type>
+          <!-- Noise is sampled independently per pixel on each frame.
+               That pixel's noise value is added to each of its color
+               channels, which at that point lie in the range [0,1]. -->
+          <mean>0.0</mean>
+          <stddev>0.007</stddev>
+        </noise>
+      </camera>
+      <plugin name="camera_controller" filename="libgazebo_ros_camera.so">
+        <alwaysOn>true</alwaysOn>
+        <updateRate>0.0</updateRate>
+        <cameraName>stereo/right</cameraName>
+        <imageTopicName>image_raw</imageTopicName>
+        <cameraInfoTopicName>camera_info</cameraInfoTopicName>
+        <frameName>camera_link_right</frameName>
+        <hackBaseline>0.07</hackBaseline>
+        <distortionK1>0.0</distortionK1>
+        <distortionK2>0.0</distortionK2>
+        <distortionK3>0.0</distortionK3>
+        <distortionT1>0.0</distortionT1>
+        <distortionT2>0.0</distortionT2>
+      </plugin>
+    </sensor>
+  </gazebo>
 </robot>

File: turtlebot3_description/urdf/turtlebot3_burger_vision.urdf.xacro (robot description, xacro)
@@ -144,58 +144,58 @@
     <child link="camera_optical_link"/>
   </joint>
-<!--  &lt;!&ndash; Camera left &ndash;&gt;-->
-<!--  <link name="camera_link_left">-->
-<!--    <collision>-->
-<!--      <origin xyz="0 0 0" rpy="0 0 0"/>-->
-<!--      <geometry>-->
-<!--        <box size="${camera_link} ${camera_link} ${camera_link}"/>-->
-<!--      </geometry>-->
-<!--    </collision>-->
-<!--    <visual>-->
-<!--      <origin xyz="0 0 0" rpy="0 0 0"/>-->
-<!--      <geometry>-->
-<!--        <box size="${camera_link} ${camera_link} ${camera_link}"/>-->
-<!--      </geometry>-->
-<!--      <material name="red"/>-->
-<!--    </visual>-->
-<!--    <inertial>-->
-<!--      <mass value="1e-5" />-->
-<!--      <origin xyz="0 0 0" rpy="0 0 0"/>-->
-<!--      <inertia ixx="1e-6" ixy="0" ixz="0" iyy="1e-6" iyz="0" izz="1e-6" />-->
-<!--    </inertial>-->
-<!--  </link>-->
-<!--  <joint name="camera_joint_left" type="fixed">-->
-<!--    <axis xyz="0 1 0" />-->
-<!--    <origin xyz="0.05 0.1 0.1" rpy="0 0 0"/>-->
-<!--    <parent link="base_link"/>-->
-<!--    <child link="camera_link_left"/>-->
-<!--  </joint>-->
-<!--  &lt;!&ndash; Camera right &ndash;&gt;-->
-<!--  <link name="camera_link_right">-->
-<!--    <collision>-->
-<!--      <origin xyz="0 0 0" rpy="0 0 0"/>-->
-<!--      <geometry>-->
-<!--        <box size="${camera_link} ${camera_link} ${camera_link}"/>-->
-<!--      </geometry>-->
-<!--    </collision>-->
-<!--    <visual>-->
-<!--      <origin xyz="0 0 0" rpy="0 0 0"/>-->
-<!--      <geometry>-->
-<!--        <box size="${camera_link} ${camera_link} ${camera_link}"/>-->
-<!--      </geometry>-->
-<!--      <material name="red"/>-->
-<!--    </visual>-->
-<!--    <inertial>-->
-<!--      <mass value="1e-5" />-->
-<!--      <origin xyz="0 0 0" rpy="0 0 0"/>-->
-<!--      <inertia ixx="1e-6" ixy="0" ixz="0" iyy="1e-6" iyz="0" izz="1e-6" />-->
-<!--    </inertial>-->
-<!--  </link>-->
-<!--  <joint name="camera_joint_right" type="fixed">-->
-<!--    <axis xyz="0 1 0" />-->
-<!--    <origin xyz="0.05 -0.1 0.1" rpy="0 0 0"/>-->
-<!--    <parent link="base_link"/>-->
-<!--    <child link="camera_link_right"/>-->
-<!--  </joint>-->
+  <!-- Camera left -->
+  <link name="camera_link_left">
+    <collision>
+      <origin xyz="0 0 0" rpy="0 0 0"/>
+      <geometry>
+        <box size="${camera_link} ${camera_link} ${camera_link}"/>
+      </geometry>
+    </collision>
+    <visual>
+      <origin xyz="0 0 0" rpy="0 0 0"/>
+      <geometry>
+        <box size="${camera_link} ${camera_link} ${camera_link}"/>
+      </geometry>
+      <material name="red"/>
+    </visual>
+    <inertial>
+      <mass value="1e-5" />
+      <origin xyz="0 0 0" rpy="0 0 0"/>
+      <inertia ixx="1e-6" ixy="0" ixz="0" iyy="1e-6" iyz="0" izz="1e-6" />
+    </inertial>
+  </link>
+  <joint name="camera_joint_left" type="fixed">
+    <axis xyz="0 1 0" />
+    <origin xyz="0.05 0.1 0.1" rpy="0 0 0"/>
+    <parent link="base_link"/>
+    <child link="camera_link_left"/>
+  </joint>
+  <!-- Camera right -->
+  <link name="camera_link_right">
+    <collision>
+      <origin xyz="0 0 0" rpy="0 0 0"/>
+      <geometry>
+        <box size="${camera_link} ${camera_link} ${camera_link}"/>
+      </geometry>
+    </collision>
+    <visual>
+      <origin xyz="0 0 0" rpy="0 0 0"/>
+      <geometry>
+        <box size="${camera_link} ${camera_link} ${camera_link}"/>
+      </geometry>
+      <material name="red"/>
+    </visual>
+    <inertial>
+      <mass value="1e-5" />
+      <origin xyz="0 0 0" rpy="0 0 0"/>
+      <inertia ixx="1e-6" ixy="0" ixz="0" iyy="1e-6" iyz="0" izz="1e-6" />
+    </inertial>
+  </link>
+  <joint name="camera_joint_right" type="fixed">
+    <axis xyz="0 1 0" />
+    <origin xyz="0.05 -0.1 0.1" rpy="0 0 0"/>
+    <parent link="base_link"/>
+    <child link="camera_link_right"/>
+  </joint>
   <joint name="imu_joint" type="fixed">
     <parent link="base_link"/>
